Commit message: pro version update

File: source/big_wave_lab/big_wave_lab/assets/robots/tienkung_robots/tienkung_pro/urdf/tiangong2.0_pro_training.urdf (robot description, URDF)
Before this commit: robot tiangong2pro_urdf, 37 links, 36 joints
Links:
- removed link left_hand
- removed link right_hand
Joints:
- removed joint left_hand_joint
- removed joint right_hand

File: source/big_wave_lab/big_wave_lab/assets/robots/tienkung_robots/tienkung_pro/urdf/tiangong2_pro_hand_extension.urdf (robot description, URDF)
Before this commit: robot tiangong2.0_pro_edit_joint_limit, 1 links, 0 joints
Links:
- removed link tiangong2pro_urdf
- added link ankle_pitch_l_link, mass 0.111609; collision mesh filename=../meshes/ankle_pitch_l_link.STL; visual mesh filename=../meshes_decimated/ankle_pitch_l_link.STL
- added link ankle_pitch_r_link, mass 0.111609; collision mesh filename=../meshes/ankle_pitch_r_link.STL; visual mesh filename=../meshes_decimated/ankle_pitch_r_link.STL
- added link ankle_roll_l_link, mass 1.017381; collision mesh filename=../meshes/ankle_roll_l_link.STL; visual mesh filename=../meshes_decimated/ankle_roll_l_link.STL
- added link ankle_roll_r_link, mass 1.017381; collision mesh filename=../meshes/ankle_roll_r_link.STL; visual mesh filename=../meshes_decimated/ankle_roll_r_link.STL
- added link body_yaw_link, mass 22.0; collision mesh filename=../meshes/body_yaw_link.STL; visual mesh filename=../meshes_decimated/body_yaw_link.STL
- added link camera_head_link, mass 0.1; collision mesh filename=../meshes/camera_head_link.STL; visual mesh filename=../meshes_decimated/camera_head_link.STL
- added link elbow_pitch_l_link, mass 0.246311; collision mesh filename=../meshes/elbow_pitch_l_link.STL; visual mesh filename=../meshes_decimated/elbow_pitch_l_link.STL
- added link elbow_pitch_r_link, mass 0.246311; collision mesh filename=../meshes/elbow_pitch_r_link.STL; visual mesh filename=../meshes_decimated/elbow_pitch_r_link.STL
- added link elbow_yaw_l_link, mass 0.986828; collision mesh filename=../meshes/elbow_yaw_l_link.STL; visual mesh filename=../meshes_decimated/elbow_yaw_l_link.STL
- added link elbow_yaw_r_link, mass 0.986828; collision mesh filename=../meshes/elbow_yaw_r_link.STL; visual mesh filename=../meshes_decimated/elbow_yaw_r_link.STL
- added link head_pitch_link, mass 0.23046; collision mesh filename=../meshes/head_pitch_link.STL; visual mesh filename=../meshes_decimated/head_pitch_link.STL
- added link head_roll_link, mass 0.844627; collision mesh filename=../meshes/head_roll_link.STL; visual mesh filename=../meshes_decimated/head_roll_link.STL
- added link head_yaw_link, mass 0.088397; collision mesh filename=../meshes/head_yaw_link.STL; visual mesh filename=../meshes_decimated/head_yaw_link.STL
- added link hip_pitch_l_link, mass 3.951912; collision mesh filename=../meshes/hip_pitch_l_link.STL; visual mesh filename=../meshes_decimated/hip_pitch_l_link.STL
- added link hip_pitch_r_link, mass 3.951912; collision mesh filename=../meshes/hip_pitch_r_link.STL; visual mesh filename=../meshes_decimated/hip_pitch_r_link.STL
- added link hip_roll_l_link, mass 0.672983; collision mesh filename=../meshes/hip_roll_l_link.STL; visual mesh filename=../meshes_decimated/hip_roll_l_link.STL
- added link hip_roll_r_link, mass 0.672983; collision mesh filename=../meshes/hip_roll_r_link.STL; visual mesh filename=../meshes_decimated/hip_roll_r_link.STL
- added link hip_yaw_l_link, mass 6.670795; collision mesh filename=../meshes/hip_yaw_l_link.STL; visual mesh filename=../meshes_decimated/hip_yaw_l_link.STL
- added link hip_yaw_r_link, mass 6.670795; collision mesh filename=../meshes/hip_yaw_r_link.STL; visual mesh filename=../meshes_decimated/hip_yaw_r_link.STL
- added link imu_link, mass 0.02; collision mesh filename=../meshes/imu_link.STL; visual mesh filename=../meshes_decimated/imu_link.STL
- added link knee_pitch_l_link, mass 2.312685; collision mesh filename=../meshes/knee_pitch_l_link.STL; visual mesh filename=../meshes_decimated/knee_pitch_l_link.STL
- added link knee_pitch_r_link, mass 2.312685; collision mesh filename=../meshes/knee_pitch_r_link.STL; visual mesh filename=../meshes_decimated/knee_pitch_r_link.STL
- added link left_hand, mass 0.131751; collision mesh filename=file:///home/cai/humanoid_ws/big_wave_lab/source/big_wave_l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 scale=1. 1. 1.; visual mesh filename=file:///home/cai/humanoid_ws/big_wave_lab/source/big_wave_l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 scale=1. 1. 1.
- added link left_tcp_link, mass 0.218186; collision mesh filename=../meshes/left_tcp_link.STL; visual mesh filename=../meshes_decimated/left_tcp_link.STL
- added link pelvis, mass 5.639; collision mesh filename=../meshes/pelvis.STL; visual mesh filename=../meshes_decimated/pelvis.STL
- added link right_hand, mass 0.131751; collision mesh filename=file:///home/cai/humanoid_ws/big_wave_lab/source/big_wave_l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 scale=1. 1. 1.; visual mesh filename=file:///home/cai/humanoid_ws/big_wave_lab/source/big_wave_l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 scale=1. 1. 1.
- added link right_tcp_link, mass 0.218186; collision mesh filename=../meshes/right_tcp_link.STL; visual mesh filename=../meshes_decimated/right_tcp_link.STL
- added link shoulder_pitch_l_link, mass 1.032698; collision mesh filename=../meshes/shoulder_pitch_l_link.STL; visual mesh filename=../meshes_decimated/shoulder_pitch_l_link.STL
- added link shoulder_pitch_r_link, mass 1.032698; collision mesh filename=../meshes/shoulder_pitch_r_link.STL; visual mesh filename=../meshes_decimated/shoulder_pitch_r_link.STL
- added link shoulder_roll_l_link, mass 0.440997; collision mesh filename=../meshes/shoulder_roll_l_link.STL; visual mesh filename=../meshes_decimated/shoulder_roll_l_link.STL
- added link shoulder_roll_r_link, mass 0.440997; collision mesh filename=../meshes/shoulder_roll_r_link.STL; visual mesh filename=../meshes_decimated/shoulder_roll_r_link.STL
- added link shoulder_yaw_l_link, mass 1.365033; collision mesh filename=../meshes/shoulder_yaw_l_link.STL; visual mesh filename=../meshes_decimated/shoulder_yaw_l_link.STL
- added link shoulder_yaw_r_link, mass 1.365033; collision mesh filename=../meshes/shoulder_yaw_r_link.STL; visual mesh filename=../meshes_decimated/shoulder_yaw_r_link.STL
- added link wrist_pitch_l_link, mass 0.262007; collision mesh filename=../meshes/wrist_pitch_l_link.STL; visual mesh filename=../meshes_decimated/wrist_pitch_l_link.STL
- added link wrist_pitch_r_link, mass 0.262007; collision mesh filename=../meshes/wrist_pitch_r_link.STL; visual mesh filename=../meshes_decimated/wrist_pitch_r_link.STL
- added link wrist_roll_l_link, mass 0.131751; collision mesh filename=../meshes/wrist_roll_l_link.STL; visual mesh filename=../meshes_decimated/wrist_roll_l_link.STL
- added link wrist_roll_r_link, mass 0.131751; collision mesh filename=../meshes/wrist_roll_r_link.STL; visual mesh filename=../meshes_decimated/wrist_roll_r_link.STL
Joints:
- added joint ankle_pitch_l_joint: type revolute, parent knee_pitch_l_link, child ankle_pitch_l_link, origin xyz=0 0 -0.4 rpy=0 0 0, axis 0 1 0, limit lower=-1.2217304763960306 upper=0.5235987755982988 effort=55.0 velocity=14.137166941154069
- added joint ankle_pitch_r_joint: type revolute, parent knee_pitch_r_link, child ankle_pitch_r_link, origin xyz=0 0.00099989 -0.4 rpy=0 0 0, axis 0 1 0, limit lower=-1.2217304763960306 upper=0.5235987755982988 effort=55.0 velocity=14.137166941154069
- added joint ankle_roll_l_joint: type revolute, parent ankle_pitch_l_link, child ankle_roll_l_link, origin xyz=0 0 0 rpy=0 0 0, axis 1 0 0, limit lower=-0.5235987755982988 upper=0.5235987755982988 effort=55.0 velocity=14.137166941154069
- added joint ankle_roll_r_joint: type revolute, parent ankle_pitch_r_link, child ankle_roll_r_link, origin xyz=0 0 0 rpy=0 0 0, axis 1 0 0, limit lower=-0.5235987755982988 upper=0.5235987755982988 effort=55.0 velocity=14.137166941154069
- added joint body_yaw_joint: type revolute, parent pelvis, child body_yaw_link, origin xyz=0 0 0 rpy=0 0 0, axis 0 0 1, limit lower=-2.9670597283903604 upper=2.9670597283903604 effort=91.0 velocity=9.215338450530059
- added joint camera_head_joint: type fixed, parent head_roll_link, child camera_head_link, origin xyz=0.075191 0.010935 0.074436 rpy=-1.8326 0 -1.5708, axis 0 0 0
- added joint elbow_pitch_l_joint: type revolute, parent shoulder_yaw_l_link, child elbow_pitch_l_link, origin xyz=0.02 0 -0.1975 rpy=0 0 0, axis 0 1 0, limit lower=-2.6179938779914944 upper=0.2617993877991494 effort=35.0 velocity=5.235987755982989
- added joint elbow_pitch_r_joint: type revolute, parent shoulder_yaw_r_link, child elbow_pitch_r_link, origin xyz=0.02 0 -0.1975 rpy=0 0 0, axis 0 1 0, limit lower=-2.6179938779914944 upper=0.2617993877991494 effort=35.0 velocity=5.235987755982989
- added joint elbow_yaw_l_joint: type revolute, parent elbow_pitch_l_link, child elbow_yaw_l_link, origin xyz=-0.02 0 -0.0543 rpy=0 0 0, axis 0 0 1, limit lower=-2.9670597283903604 upper=2.9670597283903604 effort=24.0 velocity=10.471975511965978
- added joint elbow_yaw_r_joint: type revolute, parent elbow_pitch_r_link, child elbow_yaw_r_link, origin xyz=-0.02 0 -0.0543 rpy=0 0 0, axis 0 0 1, limit lower=-2.9670597283903604 upper=2.9670597283903604 effort=24.0 velocity=10.471975511965978
- added joint head_pitch_joint: type revolute, parent head_yaw_link, child head_pitch_link, origin xyz=0.01455 0 0.0304 rpy=0 0.2618 0, axis 0 1 0, limit lower=-0.4363323129985824 upper=0.4363323129985824 effort=6.3 velocity=7.5398223686155035
- added joint head_roll_joint: type revolute, parent head_pitch_link, child head_roll_link, origin xyz=0 0 0 rpy=0 0 0, axis 1 0 0, limit lower=-0.4537856055185257 upper=0.4537856055185257 effort=6.3 velocity=7.5398223686155035
- added joint head_yaw_joint: type revolute, parent body_yaw_link, child head_yaw_link, origin xyz=-0.002 0 0.56508 rpy=0 0 0, axis 0 0 1, limit lower=-1.5707963267948966 upper=1.5707963267948966 effort=6.3 velocity=7.5398223686155035
- added joint hip_pitch_l_joint: type revolute, parent hip_roll_l_link, child hip_pitch_l_link, origin xyz=0 0.122 -0.046 rpy=0 0 0, axis 0 1 0, limit lower=-2.792526803190927 upper=2.0943951023931953 effort=330.0 velocity=15.707963267948966
- added joint hip_pitch_r_joint: type revolute, parent hip_roll_r_link, child hip_pitch_r_link, origin xyz=0 -0.122 -0.046 rpy=0 0 0, axis 0 1 0, limit lower=-2.792526803190927 upper=2.0943951023931953 effort=330.0 velocity=15.707963267948966
- added joint hip_roll_l_joint: type revolute, parent pelvis, child hip_roll_l_link, origin xyz=0 0.028 -0.0857 rpy=0 0 0, axis 1 0 0, limit lower=-0.7853981633974483 upper=0.7853981633974483 effort=235.0 velocity=16.755160819145562
- added joint hip_roll_r_joint: type revolute, parent pelvis, child hip_roll_r_link, origin xyz=0 -0.028 -0.0857 rpy=0 0 0, axis 1 0 0, limit lower=-0.7853981633974483 upper=0.7853981633974483 effort=235.0 velocity=16.755160819145562
- added joint hip_yaw_l_joint: type revolute, parent hip_pitch_l_link, child hip_yaw_l_link, origin xyz=0 -0.00015 -0.0987 rpy=0 0 0, axis 0 0 1, limit lower=-1.0471975511965976 upper=1.0471975511965976 effort=235.0 velocity=16.755160819145562
- added joint hip_yaw_r_joint: type revolute, parent hip_pitch_r_link, child hip_yaw_r_link, origin xyz=0 0 -0.0987 rpy=0 0 0, axis 0 0 1, limit lower=-1.0471975511965976 upper=1.0471975511965976 effort=235.0 velocity=16.755160819145562
- added joint imu_joint: type fixed, parent pelvis, child imu_link, origin xyz=0.0499 -0.0358 -0.03194 rpy=0 0 0, axis 0 0 0
- added joint knee_pitch_l_joint: type revolute, parent hip_yaw_l_link, child knee_pitch_l_link, origin xyz=0 0.00010715 -0.3013 rpy=0 0 0, axis 0 1 0, limit lower=0.0 upper=2.3911010752322315 effort=330.0 velocity=15.707963267948966
- added joint knee_pitch_r_joint: type revolute, parent hip_yaw_r_link, child knee_pitch_r_link, origin xyz=0 9.9938E-05 -0.3013 rpy=0 0 0, axis 0 1 0, limit lower=0.0 upper=2.3911010752322315 effort=330.0 velocity=15.707963267948966
- added joint left_hand_joint: type fixed, parent left_tcp_link, child left_hand, origin xyz=0 0 0 rpy=0 0 0, axis 0 0 0
- added joint left_tcp_joint: type fixed, parent wrist_roll_l_link, child left_tcp_link, origin xyz=0 0 -0.0848 rpy=0 0 0, axis 0 0 0
- added joint right_hand: type fixed, parent right_tcp_link, child right_hand, origin xyz=0 0 0 rpy=0 0 0, axis 0 0 0
- added joint right_tcp_joint: type fixed, parent wrist_roll_r_link, child right_tcp_link, origin xyz=0 0 -0.0848 rpy=0 0 0, axis 0 0 0
- added joint shoulder_pitch_l_joint: type revolute, parent body_yaw_link, child shoulder_pitch_l_link, origin xyz=0 0.1444 0.37712 rpy=0.087266 0 0, axis 0 1 0, limit lower=-2.9670597283903604 upper=2.9670597283903604 effort=91.0 velocity=9.215338450530059
- added joint shoulder_pitch_r_joint: type revolute, parent body_yaw_link, child shoulder_pitch_r_link, origin xyz=0 -0.1444 0.37712 rpy=-0.087266 0 0, axis 0 1 0, limit lower=-2.9670597283903604 upper=2.9670597283903604 effort=91.0 velocity=9.215338450530059
- added joint shoulder_roll_l_joint: type revolute, parent shoulder_pitch_l_link, child shoulder_roll_l_link, origin xyz=0 0.068 0 rpy=0 0 0, axis 1 0 0, limit lower=-0.2618 upper=2.6180 effort=95.0 velocity=3.979350694547071
- added joint shoulder_roll_r_joint: type revolute, parent shoulder_pitch_r_link, child shoulder_roll_r_link, origin xyz=0 -0.068 0 rpy=0 0 0, axis 1 0 0, limit lower=-2.6180 upper=0.2618 effort=95.0 velocity=3.979350694547071
- added joint shoulder_yaw_l_joint: type revolute, parent shoulder_roll_l_link, child shoulder_yaw_l_link, origin xyz=0 0 -0.1025 rpy=0 0 0, axis 0 0 1, limit lower=-2.9670597283903604 upper=2.9670597283903604 effort=35.0 velocity=5.235987755982989
- added joint shoulder_yaw_r_joint: type revolute, parent shoulder_roll_r_link, child shoulder_yaw_r_link, origin xyz=0 0 -0.1025 rpy=0 0 0, axis 0 0 1, limit lower=-2.9670597283903604 upper=2.9670597283903604 effort=35.0 velocity=5.235987755982989
- added joint wrist_pitch_l_joint: type revolute, parent elbow_yaw_l_link, child wrist_pitch_l_link, origin xyz=0 0 -0.1887 rpy=0 0 0, axis 0 1 0, limit lower=-0.7854 upper=1.1345 effort=6.3 velocity=7.5398223686155035
- added joint wrist_pitch_r_joint: type revolute, parent elbow_yaw_r_link, child wrist_pitch_r_link, origin xyz=0 0 -0.1887 rpy=0 0 0, axis 0 1 0, limit lower=-0.7854 upper=1.0472 effort=6.3 velocity=7.5398223686155035
- added joint wrist_roll_l_joint: type revolute, parent wrist_pitch_l_link, child wrist_roll_l_link, origin xyz=0 0 -0.02 rpy=0 0 0, axis 1 0 0, limit lower=-1.6581 upper=1.3090 effort=6.3 velocity=7.5398223686155035
- added joint wrist_roll_r_joint: type revolute, parent wrist_pitch_r_link, child wrist_roll_r_link, origin xyz=0 0 -0.02 rpy=0 0 0, axis 1 0 0, limit lower=-1.3090 upper=1.5708 effort=6.3 velocity=7.5398223686155035
